Commit message: working :)

File: src/arm_assembly/urdf/arm_assembly.urdf (robot description, URDF)
Before this commit: robot wroboarm_22, 7 links, 6 joints
Links:
- link base_link: mass None -> 0.93972387307473; geometry collision mesh filename=package://arm_assembly/meshes/base_link.STL; visual mesh filename=package://arm_assembly/meshes/base_link.STL
- link forarm_link: geometry collision mesh filename=package://arm_assembly/meshes/forarm_link.STL; visual mesh filename=package://arm_assembly/meshes/forarm_link.STL
- link manipulator_link: geometry collision mesh filename=package://arm_assembly/meshes/manipulator_link.STL; visual mesh filename=package://arm_assembly/meshes/manipulator_link.STL
- link shoulderBase_link: geometry collision mesh filename=package://arm_assembly/meshes/shoulderBase_link.STL; visual mesh filename=package://arm_assembly/meshes/shoulderBase_link.STL
- link upperArm_link: geometry collision mesh filename=package://arm_assembly/meshes/upperArm_link.STL; visual mesh filename=package://arm_assembly/meshes/upperArm_link.STL
- link wirstBase_link: geometry collision mesh filename=package://arm_assembly/meshes/wirstBase_link.STL; visual mesh filename=package://arm_assembly/meshes/wirstBase_link.STL
- link wrist_link: geometry collision mesh filename=package://arm_assembly/meshes/wrist_link.STL; visual mesh filename=package://arm_assembly/meshes/wrist_link.STL
Joints:
- joint elbow: limit lower=-2.26893 upper=0.174533 effort=50 velocity=1.5 -> lower=0 upper=3.1 effort=50 velocity=1.5; type revolute -> continuous
- joint forearm_roll: type revolute -> continuous
- joint shoulder: type revolute -> continuous
- joint turntable: limit lower=-0.523599 upper=1.0472 effort=50 velocity=1.5 -> lower=-3.1 upper=3.1 effort=50 velocity=1.5; type revolute -> continuous
- joint wrist_pitch: limit lower=-3.1 upper=3.1 effort=50 velocity=1.5 -> lower=-1.5707963267948966 upper=1.5707963267948966 effort=50 velocity=1.5; type revolute -> continuous
- joint wrist_roll: limit lower=-3.1 upper=3.1 effort=50 velocity=1.5 -> lower=-3.15 upper=3.15 effort=50 velocity=1.5; type revolute -> continuous

Commit message: fixed enc read bug

File: src/arm_assembly/urdf/arm_assembly.urdf (robot description, URDF)
Before this commit: robot arm_assembly, 7 links, 6 joints
Links:
- link base_link: geometry collision mesh filename=package://arm_assembly/meshes/base_link.stl; visual mesh filename=package://arm_assembly/meshes/base_link.stl
- link forarm_link: geometry collision mesh filename=package://arm_assembly/meshes/forarm_link.stl; visual mesh filename=package://arm_assembly/meshes/forarm_link.stl
- link manipulator_link: geometry collision mesh filename=package://arm_assembly/meshes/manipulator_link.stl; visual mesh filename=package://arm_assembly/meshes/manipulator_link.stl
- link shoulderBase_link: geometry collision mesh filename=package://arm_assembly/meshes/shoulderBase_link.stl; visual mesh filename=package://arm_assembly/meshes/shoulderBase_link.stl
- link upperArm_link: geometry collision mesh filename=package://arm_assembly/meshes/upperArm_link.stl; visual mesh filename=package://arm_assembly/meshes/upperArm_link.stl
- link wirstBase_link: geometry collision mesh filename=package://arm_assembly/meshes/wirstBase_link.stl; visual mesh filename=package://arm_assembly/meshes/wirstBase_link.stl
- link wrist_link: geometry collision mesh filename=package://arm_assembly/meshes/wrist_link.stl; visual mesh filename=package://arm_assembly/meshes/wrist_link.stl

File: src/wroboarm_21/urdf/wroboarm_21.urdf (robot description, URDF)
Before this commit: robot wroboarm_21, 8 links, 7 joints
Links:
- link elbow: geometry collision mesh filename=package://wroboarm_21/meshes/elbow.stl; visual mesh filename=package://wroboarm_21/meshes/elbow.stl
- link forearm: geometry collision mesh filename=package://wroboarm_21/meshes/forearm.stl; visual mesh filename=package://wroboarm_21/meshes/forearm.stl
- link gearbox: geometry collision mesh filename=package://wroboarm_21/meshes/gearbox.stl; visual mesh filename=package://wroboarm_21/meshes/gearbox.stl
- link manipulator: geometry collision mesh filename=package://wroboarm_21/meshes/manipulator.stl; visual mesh filename=package://wroboarm_21/meshes/manipulator.stl
- link turntable: geometry collision mesh filename=package://wroboarm_21/meshes/turntable.stl; visual mesh filename=package://wroboarm_21/meshes/turntable.stl
- link upperarm: geometry collision mesh filename=package://wroboarm_21/meshes/upperarm.stl; visual mesh filename=package://wroboarm_21/meshes/upperarm.stl
- link wrist: geometry collision mesh filename=package://wroboarm_21/meshes/wrist.stl; visual mesh filename=package://wroboarm_21/meshes/wrist.stl

File: src/wroboarm_22/urdf/wroboarm_22.urdf (robot description, URDF)
Before this commit: robot wroboarm_22, 7 links, 6 joints
Links:
- link base_link: geometry collision mesh filename=package://wroboarm_22/meshes/base_link.stl; visual mesh filename=package://wroboarm_22/meshes/base_link.stl
- link forarm_link: geometry collision mesh filename=package://wroboarm_22/meshes/forarm_link.stl; visual mesh filename=package://wroboarm_22/meshes/forarm_link.stl
- link manipulator_link: geometry collision mesh filename=package://wroboarm_22/meshes/manipulator_link.stl; visual mesh filename=package://wroboarm_22/meshes/manipulator_link.stl
- link shoulderBase_link: geometry collision mesh filename=package://wroboarm_22/meshes/shoulderBase_link.stl; visual mesh filename=package://wroboarm_22/meshes/shoulderBase_link.stl
- link upperArm_link: geometry collision mesh filename=package://wroboarm_22/meshes/upperArm_link.stl; visual mesh filename=package://wroboarm_22/meshes/upperArm_link.stl
- link wirstBase_link: geometry collision mesh filename=package://wroboarm_22/meshes/wirstBase_link.stl; visual mesh filename=package://wroboarm_22/meshes/wirstBase_link.stl
- link wrist_link: geometry collision mesh filename=package://wroboarm_22/meshes/wrist_link.stl; visual mesh filename=package://wroboarm_22/meshes/wrist_link.stl
