Commit message: fixin' things

File: src/wroboarm_22/urdf/wroboarm_22.urdf (robot description, URDF)
Before this commit: robot wroboarm_22, 7 links, 6 joints
Joints:
- joint elbow: limit lower=-2.26893 upper=0.174533 effort=50 velocity=1.5 -> lower=-1.57 upper=1.57 effort=50 velocity=1.5
- joint forearm_roll: limit lower=-3.1 upper=3.1 effort=50 velocity=1.5 -> lower=-1.57 upper=1.57 effort=50 velocity=1.5
- joint shoulder: limit lower=-0.349 upper=0.78539 effort=50 velocity=1.5 -> lower=-1.57 upper=1.57 effort=50 velocity=1.5
- joint turntable: limit lower=-0.523599 upper=1.0472 effort=50 velocity=1.5 -> lower=-1.57 upper=1.57 effort=50 velocity=1.5
- joint wrist_pitch: limit lower=-3.1 upper=3.1 effort=50 velocity=1.5 -> lower=-1.57 upper=1.57 effort=50 velocity=1.5
- joint wrist_roll: limit lower=-3.1 upper=3.1 effort=50 velocity=1.5 -> lower=-1.57 upper=1.57 effort=50 velocity=1.5
