Commit message: WIP on joint limits

File: src/wroboarm_23/urdf/ArmAssembly.SLDASM.urdf (robot description, URDF)
Before this commit: robot wroboarm_23, 7 links, 6 joints
Joints:
- joint elbowPitch_joint: limit (none) -> lower=0 upper=1.57 effort=50 velocity=1.5; type continuous -> revolute
- joint elbowRoll_joint: limit (none) -> lower=0 upper=1.57 effort=50 velocity=1.5; type continuous -> revolute
- joint shoulder_joint: limit (none) -> lower=0 upper=1.57 effort=50 velocity=1.5; type continuous -> revolute
- joint turntable_joint: limit (none) -> lower=0 upper=1.57 effort=50 velocity=1.5; type continuous -> revolute
- joint wristPitch_joint: limit (none) -> lower=0 upper=1.57 effort=50 velocity=1.5; type continuous -> revolute
- joint wristRoll_link: limit (none) -> lower=0 upper=1.57 effort=50 velocity=1.5; type continuous -> revolute
